File: hard/!ADDR_CNT/MUX16bitAndAddrCnt/MUX16bit.kicad_pcb (KiCad board)
At the start: 2 copper layers, 149.9 x 99.1 mm, 36 parts, among them J1 Conn_01x17_Female, J10 Conn_01x01_Male, J11 Conn_01x01_Male, J2 Conn_01x17_Female, J3 Conn_01x17_Female, J4 Conn_01x17_Female, J5 Conn_01x17_Female, J6 Conn_01x01_Male, J7 Conn_01x03_Male, J8 Screw_Terminal_01x02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

Commit message: KiCAD 5 -> 9
Connections:
- net /~E renamed /~{E}
Other:
- net class Default removed
- board text added: "~{E}"
- board text removed: "~E"
