File: hard/!ALU/AND_SMD/AND.kicad_pcb (KiCad board)
At the start: 2 copper layers, 81.3 x 27.9 mm, 10 parts, among them J1 Conn_01x08_Male, J2 Conn_01x08_Male, J3 Conn_01x08_Male, J4 Conn_01x04_Male, U1 74LS573, U2 74LS08, U3 74LS08

Commit message: KiCAD 5 -> 9
Connections:
- net /~OE renamed /~{OE}
Other:
- net class Default removed
- board text added: "~{OE}"
- board text removed: "~OE"
