File: hard/!REGS/Regs-v6/Regs-v6.kicad_pcb (KiCad board)
At the start: 2 copper layers, 160 x 99.1 mm, 59 parts, among them J1 Conn_01x22_Socket, J10 Conn_01x01_Male, J11 Conn_01x03_Male, J12 Conn_01x01_Male, J13 Conn_01x01_Male, J14 Conn_01x01_Male, J15 Conn_01x01_Male, J16 Screw_Terminal_01x02, J17 Conn_01x09_Male, J18 Conn_01x09_Male, J19 Conn_01x01_Male, J2 Conn_01x22_Socket, J20 Conn_01x01_Male, J21 Conn_01x01_Male, J22 Conn_01x01_Male, J23 Conn_01x01_Male, J24 Conn_01x01_Male, J3 Conn_01x22_Socket, J4 Conn_01x22_Socket, J5 Conn_01x22_Socket, J6 Conn_01x22_Socket, J7 Conn_01x22_Socket, J8 Conn_01x22_Socket, J9 Conn_01x01_Male, Q1 IRLML5203, U1 REG_CNT, U10 REG_CNT, U11 REG_CNT, U12 REG_CNT, U13 74LS139, U14 74HC00, U15 MUX2-1, U16 REG_CNT, U17 REG_CNT, U18 REG_CNT, U19 REG_CNT, U2 REG_CNT, U3 REG_CNT, U4 REG_CNT, U5 REG_CNT, U6 REG_CNT, U7 REG_CNT, U8 REG_CNT, U9 REG_CNT

Commit message: Regs v6.1 is ok
Parts:
- added C10: 0.1uF, Capacitor_SMD:C_0805_2012Metric_Pad1.18x1.45mm_HandSolder, B.Cu at (78.7, 67.3)
- added C5: 0.1uF, Capacitor_SMD:C_0805_2012Metric_Pad1.18x1.45mm_HandSolder, B.Cu at (25.4, 67.3)
- added C6: 0.1uF, Capacitor_SMD:C_0805_2012Metric_Pad1.18x1.45mm_HandSolder, B.Cu at (61.0, 67.3)
- added C7: 0.1uF, Capacitor_SMD:C_0805_2012Metric_Pad1.18x1.45mm_HandSolder, B.Cu at (149.9, 67.3)
- added C8: 0.1uF, Capacitor_SMD:C_0805_2012Metric_Pad1.18x1.45mm_HandSolder, B.Cu at (114.3, 67.3)
- added C9: 0.1uF, Capacitor_SMD:C_0805_2012Metric_Pad1.18x1.45mm_HandSolder, B.Cu at (96.5, 67.3)
Other:
- board text added: "19.03.26"
- board text removed: "18.03.26"
- board text removed: "Добавить конденсаторов между каждой парой регистров!"
