File: hard/!REGS/Regs-v6/Regs-v6.kicad_sch (KiCad schematic)
At the start: 60 parts, among them J1 Conn_01x15_Female, J10 Conn_01x01_Male, J11 Conn_01x03_Male, J12 Conn_01x01_Male, J13 Conn_01x01_Male, J14 Conn_01x01_Male, J15 Conn_01x01_Male, J16 Screw_Terminal_01x02, J17 Conn_01x09_Male, J18 Conn_01x09_Male, J19 Conn_01x01_Male, J2 Conn_01x15_Female, J20 Conn_01x01_Male, J21 Conn_01x01_Male, J22 Conn_01x01_Male, J23 Conn_01x01_Male, J24 Conn_01x01_Male, J3 Conn_01x15_Female, J4 Conn_01x15_Female, J5 Conn_01x15_Female, J6 Conn_01x15_Female, J7 Conn_01x15_Female, J8 Conn_01x15_Female, J9 Conn_01x01_Male, Q1 IRLML5203, U1 REG_CNT, U10 REG_CNT, U11 REG_CNT, U12 REG_CNT, U13 74LS139, U14 74HC00, U15 MUX2-1, U16 REG_CNT, U17 REG_CNT, U18 REG_CNT, U19 REG_CNT, U2 REG_CNT, U3 REG_CNT, U4 REG_CNT, U5 REG_CNT, U6 REG_CNT, U7 REG_CNT, U8 REG_CNT, U9 REG_CNT

Commit message: Regs v6.1
Parts:
- removed J1, J2, J3, J4, J5, J6, J7, J8: Conn_01x15_Female, Connector_PinSocket_2.54mm:PinSocket_1x15_P2.54mm_Vertical, symbol Connector:Conn_01x15_Female
- added J1, J2, J3, J4, J5, J6, J7, J8: Conn_01x22_Socket, Connector_PinSocket_2.54mm:PinSocket_1x22_P2.54mm_Vertical, symbol Connector:Conn_01x22_Socket
Connections:
- net R0.0: now also J1.1 (Pin_1)
- net R0.1: now also J1.4 (Pin_4)
- net R0.2: now also J1.7 (Pin_7)
- net R0.3: now also J1.10 (Pin_10)
- net R0.4: now also J1.13 (Pin_13)
- net R0.5: now also J1.16 (Pin_16)
- net R0.6: now also J1.19 (Pin_19)
- net R0.7: now also J1.22 (Pin_22)
- net R1.0: now also J2.1 (Pin_1)
- net R1.1: now also J2.4 (Pin_4)
- net R1.2: now also J2.7 (Pin_7)
- net R1.3: now also J2.10 (Pin_10)
- net R1.4: now also J2.13 (Pin_13)
- net R1.5: now also J2.16 (Pin_16)
- net R1.6: now also J2.19 (Pin_19)
- net R1.7: now also J2.22 (Pin_22)
- net R2.0: now also J3.1 (Pin_1)
- net R2.1: now also J3.4 (Pin_4)
- net R2.2: now also J3.7 (Pin_7)
- net R2.3: now also J3.10 (Pin_10)
- net R2.4: now also J3.13 (Pin_13)
- net R2.5: now also J3.16 (Pin_16)
- net R2.6: now also J3.19 (Pin_19)
- net R2.7: now also J3.22 (Pin_22)
- net R3.0: now also J4.1 (Pin_1)
- net R3.1: now also J4.4 (Pin_4)
- net R3.2: now also J4.7 (Pin_7)
- net R3.3: now also J4.10 (Pin_10)
- net R3.4: now also J4.13 (Pin_13)
- net R3.5: now also J4.16 (Pin_16)
- net R3.6: now also J4.19 (Pin_19)
- net R3.7: now also J4.22 (Pin_22)
- net R4.0: now also J5.1 (Pin_1)
- net R4.1: now also J5.4 (Pin_4)
- net R4.2: now also J5.7 (Pin_7)
- net R4.3: now also J5.10 (Pin_10)
- net R4.4: now also J5.13 (Pin_13)
- net R4.5: now also J5.16 (Pin_16)
- net R4.6: now also J5.19 (Pin_19)
- net R4.7: now also J5.22 (Pin_22)
- net R5.0: now also J6.1 (Pin_1)
- net R5.1: now also J6.4 (Pin_4)
- net R5.2: now also J6.7 (Pin_7)
- net R5.3: now also J6.10 (Pin_10)
- net R5.4: now also J6.13 (Pin_13)
- net R5.5: now also J6.16 (Pin_16)
- net R5.6: now also J6.19 (Pin_19)
- net R5.7: now also J6.22 (Pin_22)
- net R6.0: now also J7.1 (Pin_1)
- net R6.1: now also J7.4 (Pin_4)
- net R6.2: now also J7.7 (Pin_7)
- net R6.3: now also J7.10 (Pin_10)
- net R6.4: now also J7.13 (Pin_13)
- net R6.5: now also J7.16 (Pin_16)
- net R6.6: now also J7.19 (Pin_19)
- net R6.7: now also J7.22 (Pin_22)
- net R7.0: now also J8.1 (Pin_1)
- net R7.1: now also J8.4 (Pin_4)
- net R7.2: now also J8.7 (Pin_7)
- net R7.3: now also J8.10 (Pin_10)
- net R7.4: now also J8.13 (Pin_13)
- net R7.5: now also J8.16 (Pin_16)
- net R7.6: now also J8.19 (Pin_19)
- net R7.7: now also J8.22 (Pin_22)
- no-connect marks 58 -> 114
Other:
- moved on the sheet: C1, C2, C3, C4, D1, J10, J11, J12, J13, J14, J15, J16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

Commit message: Regs v6.1 in work
Parts:
- removed R2: 10k, Resistor_SMD:R_0805_2012Metric_Pad1.20x1.40mm_HandSolder, symbol Device:R
Changed lines of the file:
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@@
 	)
 	(junction
-		(at 52.07 278.13)
-		(diameter 0)
-		(color 0 0 0 0)
-	)
-	(junction
 		(at 153.67 259.08)
 		(diameter 0)
@@
 	(wire
 		(pts
-			(xy 52.07 275.59) (xy 52.07 278.13)
-		)
-		(stroke
-			(width 0)
-			(type default)
-		)
-	)
-	(wire
-		(pts
 			(xy 76.835 270.51) (xy 80.01 270.51)
 		)
@@
 					(unit 1)
 				)
-			)
-		)
-	)
-	(symbol
-		(lib_id "Device:R")
-		(at 52.07 271.78 0)
-		(unit 1)
-		(exclude_from_sim no)
-		(in_bom yes)
-		(on_board yes)
-		(dnp no)
-		(property "Reference" "R2"
-			(at 50.165 271.78 90)
-			(effects
-				(font
-					(size 1.27 1.27)
-				)
-			)
-		)
-		(property "Value" "10k"
-			(at 52.07 271.78 90)
-			(effects
-				(font
-					(size 1.27 1.27)
-				)
-			)
-		)
-		(property "Footprint" "Resistor_SMD:R_0805_2012Metric_Pad1.20x1.40mm_HandSolder"
-			(at 50.292 271.78 90)
-			(effects
-				(font
-					(size 1.27 1.27)
-				)
-				(hide yes)
-			)
-		)
-		(property "Datasheet" "~"
-			(at 52.07 271.78 0)
-			(effects
-				(font
-					(size 1.27 1.27)
-				)
-				(hide yes)
-			)
-		)
-		(property "Description" ""
-			(at 52.07 271.78 0)
-			(effects
-				(font
-					(size 1.27 1.27)
-				)
-			)
-		)
-		(pin "1"
-		)
-		(pin "2"
-		)
-		(instances
-			(project ""
-				(path "/8209534a-5d70-4acf-9a72-9345b085efc5"
-					(reference "R2")
-					(unit 1)
-				)
-			)
-		)
-	)
-	(symbol
-		(lib_id "power:VCC")
-		(at 52.07 267.97 0)
-		(unit 1)
-		(exclude_from_sim no)
-		(in_bom yes)
-		(on_board yes)
-		(dnp no)
-		(property "Reference" "#PWR05"
-			(at 52.07 271.78 0)
-			(effects
-				(font
-					(size 1.27 1.27)
-				)
-				(hide yes)
-			)
-		)
-		(property "Value" "VCC"
-			(at 52.451 263.5758 0)
-			(effects
-				(font
-					(size 1.27 1.27)
-				)
-			)
-		)
-		(property "Footprint" ""
-			(at 52.07 267.97 0)
-			(effects
-				(font
-					(size 1.27 1.27)
-				)
-				(hide yes)
-			)
-		)
-		(property "Datasheet" ""
-			(at 52.07 267.97 0)
-			(effects
-				(font
-					(size 1.27 1.27)
-				)
-				(hide yes)
-			)
-		)
-		(property "Description" ""
-			(at 52.07 267.97 0)
-			(effects
-				(font
-					(size 1.27 1.27)
-				)
-			)
-		)
-		(pin "1"
-		)
-		(instances
-			(project ""
-				(path "/8209534a-5d70-4acf-9a72-9345b085efc5"
-					(reference "#PWR05")
-					(unit 1)
-				)

Commit message: Regs v6.1 is ok
Parts:
- added C10, C5, C6, C7, C8, C9: 0.1uF, Capacitor_SMD:C_0805_2012Metric_Pad1.18x1.45mm_HandSolder, symbol Device:C
Connections:
- net GND: now also C10.2, C5.2, C6.2, C7.2, C8.2, C9.2
- net VCC: now also C10.1, C5.1, C6.1, C7.1, C8.1, C9.1
