File: hard/!REGS/Regs-v5/Regs-v5.kicad_pcb (KiCad board)
At the start: 2 copper layers, 160 x 99.1 mm, 51 parts, among them J1 Conn_01x09_Male, J11 Conn_01x03_Male, J12 Conn_01x01_Male, J13 Conn_01x01_Male, J14 Conn_01x01_Male, J15 Conn_01x01_Male, J16 Screw_Terminal_01x02, J17 Conn_01x09_Male, J18 Conn_01x09_Male, J19 Conn_01x01_Male, J2 Conn_01x09_Male, J20 Conn_01x01_Male, J3 Conn_01x09_Male, J4 Conn_01x09_Male, J5 Conn_01x09_Male, J6 Conn_01x09_Male, J7 Conn_01x09_Male, J8 Conn_01x09_Male, Q1 IRLML5203, U1 REG_CNT, U10 REG_CNT, U11 REG_CNT, U12 REG_CNT, U13 74LS139, U14 74HC00, U15 MUX2-1, U16 REG_CNT, U17 REG_CNT, U18 REG_CNT, U19 REG_CNT, U2 REG_CNT, U3 REG_CNT, U4 REG_CNT, U5 REG_CNT, U6 REG_CNT, U7 REG_CNT, U8 REG_CNT, U9 REG_CNT

Commit message: KiCAD 5 -> 9
Connections:
- net /~Bank0 renamed /~{Bank0}
- net /~Bank1 renamed /~{Bank1}
- net /~H renamed /~{H}
- net /~L renamed /~{L}
- net /~MUL renamed /~{MUL}
- net /~R0 renamed /~{R0}
- net /~R1 renamed /~{R1}
- net /~R2 renamed /~{R2}
- net /~R3 renamed /~{R3}
- net /~Res renamed /~{Res}
Other:
- net class Default removed
- board text added: "~{Bank0}"
- board text added: "~{CS}"
- board text added: "~{Col}"
- board text added: "~{MUL}"
- board text added: "~{Res}"
- board text added: "~{Row}"
- board text removed: "~Bank0"
- board text removed: "~CS"
- board text removed: "~Col"
- board text removed: "~MUL"
- board text removed: "~Res"
- board text removed: "~Row"
