File: hard/!MUL/MUL1_SMD/MUL1.kicad_sch (KiCad schematic)
At the start: 13 parts, among them J1 Conn_01x08_Male, J2 Conn_01x09_Male, J3 Conn_01x08_Male, J4 Conn_01x01_Male, J5 Conn_01x02_Male, J6 Conn_01x01_Male, U1 74LS08, U2 74LS283, U3 74LS08, U4 74LS283

Commit message: 2 DIP and 2 SO!
Parts:
- U1, U3: footprint Package_SO:SO-14_3.9x8.65mm_P1.27mm -> Package_DIP:DIP-14_W7.62mm
Changed lines of the file:
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@@
 			)
 		)
-		(property "Footprint" "Package_SO:SO-14_3.9x8.65mm_P1.27mm"
+		(property "Footprint" "Package_DIP:DIP-14_W7.62mm"
 			(at 83.82 59.69 0)
 			(effects
@@
 			)
 		)
-		(property "Footprint" "Package_SO:SO-14_3.9x8.65mm_P1.27mm"
+		(property "Footprint" "Package_DIP:DIP-14_W7.62mm"
 			(at 83.82 72.39 0)
 			(effects
@@
 			)
 		)
-		(property "Footprint" "Package_SO:SO-14_3.9x8.65mm_P1.27mm"
+		(property "Footprint" "Package_DIP:DIP-14_W7.62mm"
 			(at 83.82 85.09 0)
 			(effects
@@
 			)
 		)
-		(property "Footprint" "Package_SO:SO-14_3.9x8.65mm_P1.27mm"
+		(property "Footprint" "Package_DIP:DIP-14_W7.62mm"
 			(at 83.82 97.79 0)
 			(effects
@@
 			)
 		)
-		(property "Footprint" "Package_SO:SO-14_3.9x8.65mm_P1.27mm"
+		(property "Footprint" "Package_DIP:DIP-14_W7.62mm"
 			(at 201.93 121.92 0)
 			(effects
@@
 			)
 		)
-		(property "Footprint" "Package_SO:SO-14_3.9x8.65mm_P1.27mm"
+		(property "Footprint" "Package_DIP:DIP-14_W7.62mm"
 			(at 83.82 116.84 0)
 			(effects
@@
 			)
 		)
-		(property "Footprint" "Package_SO:SO-14_3.9x8.65mm_P1.27mm"
+		(property "Footprint" "Package_DIP:DIP-14_W7.62mm"
 			(at 83.82 129.54 0)
 			(effects
@@
 			)
 		)
-		(property "Footprint" "Package_SO:SO-14_3.9x8.65mm_P1.27mm"
+		(property "Footprint" "Package_DIP:DIP-14_W7.62mm"
 			(at 83.82 142.24 0)
 			(effects
@@
 			)
 		)
-		(property "Footprint" "Package_SO:SO-14_3.9x8.65mm_P1.27mm"
+		(property "Footprint" "Package_DIP:DIP-14_W7.62mm"
 			(at 83.82 154.94 0)
 			(effects
@@
 			)
 		)
-		(property "Footprint" "Package_SO:SO-14_3.9x8.65mm_P1.27mm"
+		(property "Footprint" "Package_DIP:DIP-14_W7.62mm"
 			(at 220.98 121.92 0)
 			(effects
