File: hard/!ROM/ROM.kicad_pcb (KiCad board)
At the start: 2 copper layers, 149.9 x 99.1 mm, 46 parts, among them J1 Conn_01x09_Male, J10 Conn_01x01_Male, J11 Conn_01x01_Male, J12 Conn_01x09_Male, J13 Conn_01x09_Male, J14 Conn_01x01_Male, J2 Conn_01x09_Male, J3 Conn_01x09_Male, J4 Screw_Terminal_01x02, J5 Conn_01x09_Male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

Commit message: KiCAD 5 -> 9
Connections:
- net /~CS renamed /~{CS}
- net /~LDI renamed /~{LDI}
- net /~RD renamed /~{RD}
Other:
- net class Default removed
- board text added: "~{CS}"
- board text added: "~{LDI}"
- board text removed: "~CS"
- board text removed: "~LDI"
