File: hard/MUX1/MUX1.kicad_pcb (KiCad board)
At the start: 2 copper layers, 58.4 x 21.3 mm, 7 parts, among them J1 Conn_01x04_Male, J2 Conn_01x04_Male, J3 Conn_01x03_Male, J4 Conn_01x02_Male, J5 Conn_01x02_Male, U1 74LS153

Commit message: KiCAD 5 -> 9
Connections:
- net /~E renamed /~{E}
Other:
- net class Default removed
- board text added: "~{E}"
- board text removed: "~E"
