File: hard/!RAM/RAM.kicad_pcb (KiCad board)
At the start: 2 copper layers, 99.1 x 99.1 mm, 32 parts, among them J1 Conn_01x09_Male, J2 Conn_01x09_Male, J3 Conn_01x09_Male, J4 Conn_01x03_Male, J5 Conn_01x08_Male, J6 Screw_Terminal_01x02, Q1 IRLML5203, U1 74LS283, U2 CY62256-70PC, U3 74LS283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

Commit message: KiCAD 5 -> 9
Connections:
- net /~CS renamed /~{CS}
- net /~CS1 renamed /~{CS1}
- net /~CS2 renamed /~{CS2}
- net /~OE renamed /~{OE}
- net /~WR renamed /~{WR}
Other:
- net class Default removed
- board text added: "~{CS}"
- board text added: "~{OE}"
- board text added: "~{WR}"
- board text removed: "~CS"
- board text removed: "~OE"
- board text removed: "~WR"
