File: hard/!ALU/CMP/CMP.kicad_pcb (KiCad board)
At the start: 2 copper layers, 81.3 x 37.1 mm, 15 parts, among them J1 Conn_01x04_Male, J2 Conn_01x08_Male, J3 Conn_01x08_Male, J4 Conn_01x08_Male, J5 Conn_01x03_Male, J6 Conn_01x03_Male, J7 Conn_01x01_Male, U1 74LS85, U2 74HC4078, U3 74LS85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

Commit message: KiCAD 5 -> 9
Other:
- net class Default removed
- board text added: "~{SRC(B}) == DST(A)"
- board text removed: "~SRC(B) == DST(A)"
