File: hard/!ALU/MOV/MOV.kicad_pcb (KiCad board)
At the start: 2 copper layers, 81.3 x 26.7 mm, 8 parts, among them J1 Conn_01x08_Male, J2 Conn_01x08_Male, J3 Conn_01x08_Male, J4 Conn_01x04_Male, U1 74LS573

Commit message: KiCAD 5 -> 9
Connections:
- net /~OE renamed /~{OE}
Other:
- net class Default removed
- board text added: "~{OE}"
- board text removed: "~OE"
