File: hard/!MUL/MUL8x8/MUL8x8.kicad_pcb (KiCad board)
At the start: 2 copper layers, 99.1 x 99.1 mm, 24 parts, among them J1 Conn_01x09_Male, J2 Conn_01x09_Male, J3 Conn_01x09_Male, J4 Conn_01x09_Male, J5 Conn_01x01_Male, J6 Screw_Terminal_01x02, Q1 IRLML5203, U1 MUL1, U10 74HC245, U2 MUL1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

Commit message: KiCAD 5 -> 9
Connections:
- net /~MUL renamed /~{MUL}
Other:
- net class Default removed
- board text added: "~{MUL}"
- board text removed: "~MUL"

Commit message: Fix silk
Other:
- board text added: "01.05.2026"
- board text removed: "13.08.2024"
Changed lines of the file:
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@@
 		(0 "F.Cu" signal)
 		(2 "B.Cu" signal)
-		(9 "F.Adhes" user)
-		(11 "B.Adhes" user)
+		(9 "F.Adhes" user "F.Adhesive")
+		(11 "B.Adhes" user "B.Adhesive")
 		(13 "F.Paste" user)
 		(15 "B.Paste" user)
-		(5 "F.SilkS" user)
-		(7 "B.SilkS" user)
+		(5 "F.SilkS" user "F.Silkscreen")
+		(7 "B.SilkS" user "B.Silkscreen")
 		(1 "F.Mask" user)
 		(3 "B.Mask" user)
-		(17 "Dwgs.User" user)
-		(19 "Cmts.User" user)
-		(21 "Eco1.User" user)
-		(23 "Eco2.User" user)
+		(17 "Dwgs.User" user "User.Drawings")
+		(19 "Cmts.User" user "User.Comments")
+		(21 "Eco1.User" user "User.Eco1")
+		(23 "Eco2.User" user "User.Eco2")
 		(25 "Edge.Cuts" user)
 		(27 "Margin" user)
-		(31 "F.CrtYd" user)
-		(29 "B.CrtYd" user)
+		(31 "F.CrtYd" user "F.Courtyard")
+		(29 "B.CrtYd" user "B.Courtyard")
 		(35 "F.Fab" user)
 		(33 "B.Fab" user)
@@
 		)
 		(property "Value" "Conn_01x09_Male"
-			(at 0 22.65 0)
+			(at 1.33 11.46 90)
 			(layer "F.Fab")
 			(effects
@@
 		)
 		(property "Value" "Conn_01x09_Male"
-			(at 0 22.65 0)
+			(at 1.27 10.795 90)
 			(layer "F.Fab")
 			(effects
@@
 		)
 		(property "Value" "Screw_Terminal_01x02"
-			(at 2.5 5.66 0)
+			(at 2.5 3.81 0)
 			(layer "F.Fab")
 			(effects
@@
 		(layer "Edge.Cuts")
 	)
-	(gr_text "13.08.2024"
+	(gr_text "01.05.2026"
 		(at 104.775 55.88 90)
 		(layer "B.Cu")
@@
 		)
 	)
-	(gr_text "OUT\nL"
-		(at 15.24 103.505 0)
+	(gr_text "OUT L"
+		(at 17.145 102.235 0)
 		(layer "F.SilkS")
 		(effects
@@
 		)
 	)
-	(gr_text "OUT\nH"
-		(at 108.585 97.79 0)
+	(gr_text "OUT H"
+		(at 106.68 96.52 0)
 		(layer "F.SilkS")
 		(effects
@@
 		)
 	)
+	(gr_text "74HCPU"
+		(at 53.34 109.855 0)
+		(layer "F.SilkS")
+		(effects
+			(font
+				(size 1.5 1.5)
+				(thickness 0.3)
+				(bold yes)
+			)
+			(justify left bottom)
+		)
+	)

Commit message: Polishing MUL
Parts:
- removed R2: 10k, Resistor_SMD:R_0805_2012Metric_Pad1.20x1.40mm_HandSolder
- removed U8: CMD, CommonLibrary:CMD
- added U11: CMD1, Common:CMDwoC, F.Cu at (36.2, 24.1)
- U1, U2, U3, U4, U5, U6, U7: footprint CommonLibrary:MUL1 -> Common:MUL1
Routing:
- net Net-(R2-Pad1): track 4.34 -> 0.00 mm
- net VCC: track 139.1 -> 135.1 mm
Other:
- board text added: "0"
- board text added: "15"
- board text added: "15.05.2026"
- board text added: "7"
- board text added: "8"
- board text added: "AND"
- board text added: "MUL1"
- board text removed: "01.05.2026"
