File: hard/!MUL/MUL8x8/MUL8x8.kicad_sch (KiCad schematic)
At the start: 24 parts, among them J1 Conn_01x09_Male, J2 Conn_01x09_Male, J3 Conn_01x09_Male, J4 Conn_01x09_Male, J5 Conn_01x01_Male, J6 Screw_Terminal_01x02, Q1 IRLML5203, U1 MUL1, U10 74HC245, U2 MUL1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

Commit message: Polishing MUL
Parts:
- removed R2: 10k, Resistor_SMD:R_0805_2012Metric_Pad1.20x1.40mm_HandSolder, symbol Device:R
- removed U8: CMD, CommonLibrary:CMD, symbol CommonLibrary:CMD
- added U11: CMD1, Common:CMDwoC, symbol Common:CMD1
- U1, U2, U3, U4, U5, U6, U7: footprint CommonLibrary:MUL1 -> Common:MUL1
Connections:
- net A0: now also U11.1 (B0)
- net A1: now also U11.2 (B1)
- net A2: now also U11.3 (B2)
- net A3: now also U11.4 (B3)
- net A4: now also U11.5 (B4)
- net A5: now also U11.6 (B5)
- net A6: now also U11.7 (B6)
- net A7: now also U11.8 (B7)
- net B0: now also U11.10 (A1), U11.11 (A2), U11.12 (A3), U11.13 (A4), U11.14 (A5), U11.15 (A6), U11.16 (A7), U11.9 (A0)
- net GND: now also U11.27 (Gnd), U11.28 (~{OE})
- net P0: now also U11.17 (O0)
- net VCC: now also U11.26 (Vcc)
- net at U1.10 (P0): now also U11.18 (O1)
- net at U1.11 (P1): now also U11.19 (O2)
- net at U1.12 (P2): now also U11.20 (O3)
- net at U1.13 (P3): now also U11.21 (O4)
- net at U1.14 (P4): now also U11.22 (O5)
- net at U1.15 (P5): now also U11.23 (O6)
- net at U1.16 (P6): now also U11.24 (O7)
- net at R1.2: now also U11.25 (Latch)
