File: hard/!ALU/ADD/ADD.kicad_pcb (KiCad board)
At the start: 2 copper layers, 83.8 x 39.4 mm, 16 parts, among them J1 Conn_01x08_Male, J2 Conn_01x08_Male, J3 Conn_01x08_Male, J4 Conn_01x05_Male, J5 Conn_01x01_Male, J6 Conn_01x01_Male, J7 Conn_01x01_Male, U1 74LS283, U2 74LS283, U3 74LS573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

Commit message: KiCAD 5 -> 9
Connections:
- net /~(ADD_COUT&OE) renamed /~{(ADD_COUT&OE})
- net /~OE renamed /~{OE}
Other:
- net class Default removed
- board text added: "~{OE}"
- board text removed: "~OE"

Commit message: Polishing ADD
Parts:
- R3: moved to F.Cu
- moved D1 3.62 mm to (138.7, 54.6), turned to 180 degrees
- moved R1 2.70 mm to (139.7, 60.6)
- moved R3 2.61 mm to (142.2, 61.6)
- moved R2 1.91 mm to (129.5, 62.0)
Connections:
- J4 pad 1: /~{OE} -> /UseCF
- J4 pad 2: /UseCF -> /~{OE}
Routing:
- net /UseCF: track 55.5 -> 48.6 mm
- net VCC: track 116.7 -> 112.0 mm
- net /auxiliary_carry: track 81.5 -> 77.3 mm
- net Net-(D1-K): track 2.42 -> 5.08 mm
- net /~{OE}: track 45.0 -> 43.0 mm
- net /ADD_CIN: track 20.5 -> 18.6 mm
- net /Latch: track 43.1 -> 44.6 mm
- net Net-(U2-S3): track 55.8 -> 55.1 mm
Other:
- board text added: "15.05.2026"
- board text removed: "06.07.2023"
