File: hard/!ALU/ADD/ADD.kicad_sch (KiCad schematic)
At the start: 16 parts, among them J1 Conn_01x08_Male, J2 Conn_01x08_Male, J3 Conn_01x08_Male, J4 Conn_01x05_Male, J5 Conn_01x01_Male, J6 Conn_01x01_Male, J7 Conn_01x01_Male, U1 74LS283, U2 74LS283, U3 74LS573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

Commit message: Polishing ADD
Connections:
- net UseCF: now also J4.1 (Pin_1); no longer J4.2 (Pin_2)
- net ~{OE}: now also J4.2 (Pin_2); no longer J4.1 (Pin_1)
Changed lines of the file:
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@@
 	)
 	(label "UseCF"
-		(at 30.48 134.62 0)
+		(at 30.48 137.16 0)
 		(effects
 			(font
@@
 	)
 	(label "~{OE}"
-		(at 30.48 137.16 0)
+		(at 30.48 134.62 0)
 		(effects
 			(font
@@
 		)
 		(property "Value" "Conn_01x05_Male"
-			(at 28.1432 139.446 0)
-			(effects
-				(font
+			(at 23.495 131.953 90)
+			(effects
+				(font
