File: hard/!MUL/MUL1/MUL1.kicad_pcb (KiCad board)
At the start: 2 copper layers, 83.8 x 36.2 mm, 13 parts, among them J1 Conn_01x08_Male, J2 Conn_01x09_Male, J3 Conn_01x08_Male, J4 Conn_01x01_Male, J5 Conn_01x02_Male, J6 Conn_01x01_Male, U1 74LS08, U2 74LS283, U3 74LS08, U4 74LS283

Commit message: KiCAD 5 -> 9
Other:
- net class Default removed

Commit message: Polishing MUL1
Parts:
- moved R1 6.09 mm to (120.4, 76.5), turned to 0 degrees
Routing:
- net Net-(J6-Pad1): track 7.34 -> 10.9 mm
- net GND: track 140.1 -> 138.9 mm
- net /P5: track 35.1 -> 36.2 mm
- net /P3: track 30.7 -> 31.5 mm
- net /P4: track 32.2 -> 33.0 mm
Other:
- board text added: "15.05.2026"
- board text removed: "13.05.2023"
