File: hard/!Ports/Ports/Ports.kicad_pcb (KiCad board)
At the start: 2 copper layers, 99.1 x 99.1 mm, 79 parts, among them J1 Conn_01x09_Male, J2 Conn_01x09_Male, J3 Conn_01x09_Male, J4 Screw_Terminal_01x02, J5 Conn_01x04_Male, J6 Conn_01x09_Male, J7 Conn_01x02_Male, J8 Conn_01x08_Male, J9 Conn_01x02_Male, Q1 IRLML2060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

Commit message: KiCAD 5 -> 9
Other:
- net class Default removed
- board text added: "R/~{W}"
- board text added: "~{OE}"
- board text removed: "R/~W"
- board text removed: "~OE"
