File: hard/!ALU/LSR/LSR.kicad_pcb (KiCad board)
At the start: 2 copper layers, 61 x 26.7 mm, 11 parts, among them J1 Conn_01x01_Male, J2 Conn_01x08_Male, J3 Conn_01x08_Male, J4 Conn_01x01_Male, J5 Conn_01x05_Male, U1 74HC00, U2 74LS573

Commit message: KiCAD 5 -> 9
Connections:
- net /~(CF&OE) renamed /~{(CF&OE})
- net /~OE renamed /~{OE}
Other:
- net class Default removed
- board text added: "~{OE}"
- board text removed: "~OE"
